Commit message: sim2real

File: ros_ws/src/urdf_test_node/urdf/sekirei_moveit.urdf (robot description, URDF)
Before this commit: robot sekirei, 10 links, 9 joints
Joints:
- joint arm_joint1: axis 0 0 1 -> 0 0 -1
- joint arm_joint3: axis 0 1 0 -> 0 -1 0; limit lower=0 upper=3.14 effort=5 velocity=1.571 -> lower=-3.14 upper=3.14 effort=5 velocity=1.571
- joint arm_joint4: limit lower=-4.71 upper=0 effort=5 velocity=1.571 -> lower=-3.14 upper=3.14 effort=5 velocity=1.571

Commit message: sim2real

File: ros_ws/src/urdf_test_node/urdf/sekirei_moveit.urdf (robot description, URDF)
Before this commit: robot sekirei, 10 links, 9 joints
Joints:
- joint arm_joint1: axis 0 0 -1 -> 0 0 1
- joint arm_joint3: axis 0 -1 0 -> 0 1 0
