Commit message: fix: transmission ?

File: ros_ws/src/sekirei_moveit_config/urdf/sekirei_moveit.xacro (robot description, xacro)
@@ -1,3 +1,3 @@
-<?xml version="1.0"?>
+<?xml version="1.0" ?>
 <!-- 実機制御用のURDF -->
 <robot xmlns:xacro="http://ros.org/wiki/xacro" name="sekirei">
@@ -6,8 +6,15 @@
     <link name="base_link">
         <inertial>
-            <mass value="1.0"/>
-            <origin xyz="0 0 0"/>
+            <mass value="1.0" />
+            <origin xyz="0 0 0" />
             <!-- 慣性テンソル -->
-            <inertia ixx="0.01" ixy="0.0" ixz="0.0" iyy="0.01" iyz="0.0" izz="0.01"/>
+            <inertia
+                ixx="0.01"
+                ixy="0.0"
+                ixz="0.0"
+                iyy="0.01"
+                iyz="0.0"
+                izz="0.01"
+            />
         </inertial>
     </link>
@@ -16,27 +23,36 @@
         <visual>
             <geometry>
-                <mesh filename="package://robot_model/meshes/r_a_2019_2020_asm1.STL"/>
-            </geometry>
-            <origin xyz="-0.08 -0.081 0" rpy="1.57 0 0"/>
-            <material name="white">
-                <color rgba="1 1 1 1"/>
-            </material>
-        </visual>
-        <collision>
-            <geometry>
-                <cylinder length="0.1" radius="0.05"/>
-            </geometry>
-            <origin xyz="0 0 0.05" rpy="0 0 0"/>
-        </collision>
-        <inertial>
-            <mass value="0.5"/>
-            <origin xyz="0 0 0.05"/>
-            <inertia ixx="0.001" ixy="0.0" ixz="0.0" iyy="0.001" iyz="0.0" izz="0.001"/>
+                <mesh
+                    filename="package://robot_model/meshes/r_a_2019_2020_asm1.STL"
+                />
+            </geometry>
+            <origin xyz="-0.08 -0.081 0" rpy="1.57 0 0" />
+            <material name="white">
+                <color rgba="1 1 1 1" />
+            </material>
+        </visual>
+        <collision>
+            <geometry>
+                <cylinder length="0.1" radius="0.05" />
+            </geometry>
+            <origin xyz="0 0 0.05" rpy="0 0 0" />
+        </collision>
+        <inertial>
+            <mass value="0.5" />
+            <origin xyz="0 0 0.05" />
+            <inertia
+                ixx="0.001"
+                ixy="0.0"
+                ixz="0.0"
+                iyy="0.001"
+                iyz="0.0"
+                izz="0.001"
+            />
         </inertial>
     </link>
     <joint name="arm_base_link_joint" type="fixed">
-        <origin xyz="0.2 0 0.1" rpy="0 0 0"/>
-        <parent link="base_link"/>
-        <child link="arm_base_link"/>
+        <origin xyz="0.2 0 0.1" rpy="0 0 0" />
+        <parent link="base_link" />
+        <child link="arm_base_link" />
     </joint>
     <!-- Arm Link 1 -->
@@ -44,29 +60,38 @@
         <visual>
             <geometry>
-                <mesh filename="package://robot_model/meshes/r_a_2019_2020_asm2.STL"/>
-            </geometry>
-            <origin xyz="0 0 0.004" rpy="1.57 0 0"/>
-            <material name="white">
-                <color rgba="1 1 1 1"/>
-            </material>
-        </visual>
-        <collision>
-            <geometry>
-                <cylinder length="0.08" radius="0.04"/>
-            </geometry>
-            <origin xyz="0 0 0.04" rpy="0 0 0"/>
-        </collision>
-        <inertial>
-            <mass value="0.3"/>
-            <origin xyz="0 0 0.04"/>
-            <inertia ixx="0.0008" ixy="0.0" ixz="0.0" iyy="0.0008" iyz="0.0" izz="0.0002"/>
+                <mesh
+                    filename="package://robot_model/meshes/r_a_2019_2020_asm2.STL"
+                />
+            </geometry>
+            <origin xyz="0 0 0.004" rpy="1.57 0 0" />
+            <material name="white">
+                <color rgba="1 1 1 1" />
+            </material>
+        </visual>
+        <collision>
+            <geometry>
+                <cylinder length="0.08" radius="0.04" />
+            </geometry>
+            <origin xyz="0 0 0.04" rpy="0 0 0" />
+        </collision>
+        <inertial>
+            <mass value="0.3" />
+            <origin xyz="0 0 0.04" />
+            <inertia
+                ixx="0.0008"
+                ixy="0.0"
+                ixz="0.0"
+                iyy="0.0008"
+                iyz="0.0"
+                izz="0.0002"
+            />
         </inertial>
     </link>
     <joint name="arm_joint1" type="revolute">
-        <origin xyz="0 0 0" rpy="0 0 0"/>
-        <axis xyz="0 0 1"/>
-        <parent link="arm_base_link"/>
-        <child link="arm1_link"/>
-        <limit effort="5" lower="-3.14" upper="3.14" velocity="1.571"/>
+        <origin xyz="0 0 0" rpy="0 0 0" />
+        <axis xyz="0 0 1" />
+        <parent link="arm_base_link" />
+        <child link="arm1_link" />
+        <limit effort="5" lower="-3.14" upper="3.14" velocity="1.571" />
     </joint>
     <!-- Arm Link 2 -->
@@ -74,29 +99,38 @@
         <visual>
             <geometry>
-                <mesh filename="package://robot_model/meshes/r_a_2019_2020_asm3.STL"/>
-            </geometry>
-            <origin xyz="0 0 0" rpy="1.57 0 0"/>
-            <material name="white">
-                <color rgba="1 1 1 1"/>
-            </material>
-        </visual>
-        <collision>
-            <geometry>
-                <box size="0.45 0.08 0.08"/>
-            </geometry>
-            <origin xyz="0.225 0 0" rpy="0 0 0"/>
-        </collision>
-        <inertial>
-            <mass value="0.6"/>
-            <origin xyz="0.225 0 0"/>
-            <inertia ixx="0.001" ixy="0.0" ixz="0.0" iyy="0.010" iyz="0.0" izz="0.010"/>
+                <mesh
+                    filename="package://robot_model/meshes/r_a_2019_2020_asm3.STL"
+                />
+            </geometry>
+            <origin xyz="0 0 0" rpy="1.57 0 0" />
+            <material name="white">
+                <color rgba="1 1 1 1" />
+            </material>
+        </visual>
+        <collision>
+            <geometry>
+                <box size="0.45 0.08 0.08" />
+            </geometry>
+            <origin xyz="0.225 0 0" rpy="0 0 0" />
+        </collision>
+        <inertial>
+            <mass value="0.6" />
+            <origin xyz="0.225 0 0" />
+            <inertia
+                ixx="0.001"
+                ixy="0.0"
+                ixz="0.0"
+                iyy="0.010"
+                iyz="0.0"
+                izz="0.010"
+            />
         </inertial>
     </link>
     <joint name="arm_joint2" type="revolute">
-        <origin xyz="0 -0.048 0.078" rpy="0 0 0"/>
-        <axis xyz="0 1 0"/>
-        <parent link="arm1_link"/>
-        <child link="arm2_link"/>
-        <limit effort="5" lower="-3.14" upper="3.14" velocity="1.571"/>
+        <origin xyz="0 -0.048 0.078" rpy="0 0 0" />
+        <axis xyz="0 1 0" />
+        <parent link="arm1_link" />
+        <child link="arm2_link" />
+        <limit effort="5" lower="-3.14" upper="3.14" velocity="1.571" />
     </joint>
     <!-- Arm Link 3 -->
@@ -104,30 +138,39 @@
         <visual>
             <geometry>
-                <mesh filename="package://robot_model/meshes/r_a_2019_2020_asm4.STL"/>
-            </geometry>
-            <origin xyz="0 0 0" rpy="1.57 0 0"/>
-            <material name="white">
-                <color rgba="1 1 1 1"/>
-            </material>
-        </visual>
-        <collision>
-            <geometry>
-                <box size="0.5 0.08 0.08"/>
-            </geometry>
-            <origin xyz="-0.25 0 0" rpy="0 0 0"/>
-        </collision>
-        <inertial>
-            <mass value="0.5"/>
-            <origin xyz="-0.25 0 0"/>
-            <inertia ixx="0.001" ixy="0.0" ixz="0.0" iyy="0.010" iyz="0.0" izz="0.010"/>
+                <mesh
+                    filename="package://robot_model/meshes/r_a_2019_2020_asm4.STL"
+                />
+            </geometry>
+            <origin xyz="0 0 0" rpy="1.57 0 0" />
+            <material name="white">
+                <color rgba="1 1 1 1" />
+            </material>
+        </visual>
+        <collision>
+            <geometry>
+                <box size="0.5 0.08 0.08" />
+            </geometry>
+            <origin xyz="-0.25 0 0" rpy="0 0 0" />
+        </collision>
+        <inertial>
+            <mass value="0.5" />
+            <origin xyz="-0.25 0 0" />
+            <inertia
+                ixx="0.001"
+                ixy="0.0"
+                ixz="0.0"
+                iyy="0.010"
+                iyz="0.0"
+                izz="0.010"
+            />
         </inertial>
     </link>
     <!-- は？？？ -->
     <joint name="arm_joint3" type="revolute">
-        <origin xyz="0.45 0.007 0.084" rpy="0 0 0"/>
-        <axis xyz="0 1 0"/>
-        <parent link="arm2_link"/>
-        <child link="arm3_link"/>
-        <limit effort="5" lower="0" upper="3.14" velocity="1.571"/>
+        <origin xyz="0.45 0.007 0.084" rpy="0 0 0" />
+        <axis xyz="0 1 0" />
+        <parent link="arm2_link" />
+        <child link="arm3_link" />
+        <limit effort="5" lower="0" upper="3.14" velocity="1.571" />
     </joint>
     <!-- Arm Link 4 -->
@@ -135,29 +178,38 @@
         <visual>
             <geometry>
-                <mesh filename="package://robot_model/meshes/r_a_2019_2020_asm5.STL"/>
-            </geometry>
-            <origin xyz="0 0 0" rpy="1.57 3.14 0"/>
-            <material name="white">
-                <color rgba="1 1 1 1"/>
-            </material>
-        </visual>
-        <collision>
-            <geometry>
-                <cylinder length="0.08" radius="0.03"/>
-            </geometry>
-            <origin xyz="0 0 0.04" rpy="0 0 0"/>
-        </collision>
-        <inertial>
-            <mass value="0.2"/>
-            <origin xyz="0 0 0.04"/>
-            <inertia ixx="0.0005" ixy="0.0" ixz="0.0" iyy="0.0005" iyz="0.0" izz="0.0001"/>
+                <mesh
+                    filename="package://robot_model/meshes/r_a_2019_2020_asm5.STL"
+                />
+            </geometry>
+            <origin xyz="0 0 0" rpy="1.57 3.14 0" />
+            <material name="white">
+                <color rgba="1 1 1 1" />
+            </material>
+        </visual>
+        <collision>
+            <geometry>
+                <cylinder length="0.08" radius="0.03" />
+            </geometry>
+            <origin xyz="0 0 0.04" rpy="0 0 0" />
+        </collision>
+        <inertial>
+            <mass value="0.2" />
+            <origin xyz="0 0 0.04" />
+            <inertia
+                ixx="0.0005"
+                ixy="0.0"
+                ixz="0.0"
+                iyy="0.0005"
+                iyz="0.0"
+                izz="0.0001"
+            />
         </inertial>
     </link>
     <joint name="arm_joint4" type="revolute">
-        <origin xyz="-0.5 0.012 0" rpy="0 0 0"/>
-        <axis xyz="0 1 0"/>
-        <parent link="arm3_link"/>
-        <child link="arm4_link"/>
-        <limit effort="5" lower="-3.14" upper="3.14" velocity="1.571"/>
+        <origin xyz="-0.5 0.012 0" rpy="0 0 0" />
+        <axis xyz="0 1 0" />
+        <parent link="arm3_link" />
+        <child link="arm4_link" />
+        <limit effort="5" lower="-3.14" upper="3.14" velocity="1.571" />
     </joint>
     <!-- Arm Link 5 -->
@@ -165,29 +217,38 @@
         <visual>
             <geometry>
-                <mesh filename="package://robot_model/meshes/r_a_2019_l_asm6.STL"/>
-            </geometry>
-            <origin xyz="0 0 0" rpy="1.57 3.14 0"/>
-            <material name="white">
-                <color rgba="1 1 1 1"/>
-            </material>
-        </visual>
-        <collision>
-            <geometry>
-                <cylinder length="0.06" radius="0.025"/>
-            </geometry>
-            <origin xyz="0 0 0.03" rpy="0 0 0"/>
-        </collision>
-        <inertial>
-            <mass value="0.1"/>
-            <origin xyz="0 0 0.03"/>
-            <inertia ixx="0.0002" ixy="0.0" ixz="0.0" iyy="0.0002" iyz="0.0" izz="0.0001"/>
+                <mesh
+                    filename="package://robot_model/meshes/r_a_2019_l_asm6.STL"
+                />
+            </geometry>
+            <origin xyz="0 0 0" rpy="1.57 3.14 0" />
+            <material name="white">
+                <color rgba="1 1 1 1" />
+            </material>
+        </visual>
+        <collision>
+            <geometry>
+                <cylinder length="0.06" radius="0.025" />
+            </geometry>
+            <origin xyz="0 0 0.03" rpy="0 0 0" />
+        </collision>
+        <inertial>
+            <mass value="0.1" />
+            <origin xyz="0 0 0.03" />
+            <inertia
+                ixx="0.0002"
+                ixy="0.0"
+                ixz="0.0"
+                iyy="0.0002"
+                iyz="0.0"
+                izz="0.0001"
+            />
         </inertial>
     </link>
     <joint name="arm_joint5" type="revolute">
-        <origin xyz="0.06525 0.028 0.029647" rpy="0 0 0"/>
-        <axis xyz="0 0 1"/>
-        <parent link="arm4_link"/>
-        <child link="arm5_link"/>
-        <limit effort="5" lower="-1.57" upper="1.57" velocity="1.571"/>
+        <origin xyz="0.06525 0.028 0.029647" rpy="0 0 0" />
+        <axis xyz="0 0 1" />
+        <parent link="arm4_link" />
+        <child link="arm5_link" />
+        <limit effort="5" lower="-1.57" upper="1.57" velocity="1.571" />
     </joint>
     <!-- Arm Link 6 -->
@@ -195,29 +256,38 @@
         <visual>
             <geometry>
-                <mesh filename="package://robot_model/meshes/r_a_2019_l_asm7_ver2.STL"/>
-            </geometry>
-            <origin xyz="0 0 0" rpy="0 3.14 0"/>
-            <material name="white">
-                <color rgba="1 1 1 1"/>
-            </material>
-        </visual>
-        <collision>
-            <geometry>
-                <cylinder length="0.05" radius="0.02"/>
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