Commit message: add arm_hard_control

File: ros_ws/src/robot_model/urdf/sekirei.urdf (robot description, URDF)
Before this commit: robot sekirei, 10 links, 9 joints
Links:
- link arm1_link: geometry visual mesh filename=package://robot_model/meshes/r_a_2019_2020_asm2.STL
- link arm2_link: geometry visual mesh filename=package://robot_model/meshes/r_a_2019_2020_asm3.STL
- link arm3_link: geometry visual mesh filename=package://robot_model/meshes/r_a_2019_2020_asm4.STL
- link arm4_link: geometry visual mesh filename=package://robot_model/meshes/r_a_2019_2020_asm5.STL
- link arm5_link: geometry visual mesh filename=package://robot_model/meshes/r_a_2019_l_asm6.STL
- link arm6_link: geometry visual mesh filename=package://robot_model/meshes/r_a_2019_l_asm7_ver2.STL
- link arm_base_link: geometry visual mesh filename=package://robot_model/meshes/r_a_2019_2020_asm1.STL
- link gui_d435_link: geometry visual mesh filename=package://robot_model/meshes/d435.STL
- link gui_t265_link: geometry visual mesh filename=package://robot_model/meshes/t265.STL
