Commit message: add end_effector_control_node

File: ros_ws/src/robot_model/urdf/y_sekirei_moveit.xacro (robot description, xacro)
@@ -130,5 +130,5 @@
     <!-- は？？？ -->
     <joint name="arm_joint3" type="revolute">
-        <origin xyz="0.45 0.007 0.084" rpy="0 0 0"/>
+        <origin xyz="0.45 0.0 0.084" rpy="0 0 0"/>
         <axis xyz="0 1 0"/>
         <parent link="arm2_link"/>
@@ -220,5 +220,5 @@
     </link>
     <joint name="arm_joint6" type="revolute">
-        <origin xyz="0.07425 0 -0.03" rpy="0 0 0"/>
+        <origin xyz="0 0 0" rpy="0 0 0"/>
         <axis xyz="1 0 0"/>
         <parent link="arm5_link"/>
