Commit message: dummyと実機用のurdfをxacroにまとめて動作確認をした

File: ros_ws/src/robot_model/urdf/sekirei_moveit.xacro (robot description, xacro)
@@ -16,5 +16,5 @@
         <visual>
             <geometry>
-                <mesh filename="package://urdf_test_node/meshes/r_a_2019_2020_asm1.STL"/>
+                <mesh filename="package://robot_model/meshes/r_a_2019_2020_asm1.STL"/>
             </geometry>
             <origin xyz="-0.08 -0.081 0" rpy="1.57 0 0"/>
@@ -44,5 +44,5 @@
         <visual>
             <geometry>
-                <mesh filename="package://urdf_test_node/meshes/r_a_2019_2020_asm2.STL"/>
+                <mesh filename="package://robot_model/meshes/r_a_2019_2020_asm2.STL"/>
             </geometry>
             <origin xyz="0 0 0.004" rpy="1.57 0 0"/>
@@ -74,5 +74,5 @@
         <visual>
             <geometry>
-                <mesh filename="package://urdf_test_node/meshes/r_a_2019_2020_asm3.STL"/>
+                <mesh filename="package://robot_model/meshes/r_a_2019_2020_asm3.STL"/>
             </geometry>
             <origin xyz="0 0 0" rpy="1.57 0 0"/>
@@ -98,5 +98,5 @@
         <parent link="arm1_link"/>
         <child link="arm2_link"/>
-        <limit effort="5" lower="-3.14" upper="0" velocity="1.571"/>
+        <limit effort="5" lower="-3.14" upper="3.14" velocity="1.571"/>
     </joint>
     <!-- Arm Link 3 -->
@@ -104,5 +104,5 @@
         <visual>
             <geometry>
-                <mesh filename="package://urdf_test_node/meshes/r_a_2019_2020_asm4.STL"/>
+                <mesh filename="package://robot_model/meshes/r_a_2019_2020_asm4.STL"/>
             </geometry>
             <origin xyz="0 0 0" rpy="1.57 0 0"/>
@@ -128,5 +128,5 @@
         <parent link="arm2_link"/>
         <child link="arm3_link"/>
-        <limit effort="5" lower="-3.14" upper="3.14" velocity="1.571"/>
+        <limit effort="5" lower="0" upper="3.14" velocity="1.571"/>
     </joint>
     <!-- Arm Link 4 -->
@@ -134,5 +134,5 @@
         <visual>
             <geometry>
-                <mesh filename="package://urdf_test_node/meshes/r_a_2019_2020_asm5.STL"/>
+                <mesh filename="package://robot_model/meshes/r_a_2019_2020_asm5.STL"/>
             </geometry>
             <origin xyz="0 0 0" rpy="1.57 3.14 0"/>
@@ -164,5 +164,5 @@
         <visual>
             <geometry>
-                <mesh filename="package://urdf_test_node/meshes/r_a_2019_l_asm6.STL"/>
+                <mesh filename="package://robot_model/meshes/r_a_2019_l_asm6.STL"/>
             </geometry>
             <origin xyz="0 0 0" rpy="1.57 3.14 0"/>
@@ -194,5 +194,5 @@
         <visual>
             <geometry>
-                <mesh filename="package://urdf_test_node/meshes/r_a_2019_l_asm7_ver2.STL"/>
+                <mesh filename="package://robot_model/meshes/r_a_2019_l_asm7_ver2.STL"/>
             </geometry>
             <origin xyz="0 0 0" rpy="0 3.14 0"/>
@@ -224,5 +224,5 @@
         <visual>
             <geometry>
-                <mesh filename="package://urdf_test_node/meshes/d435.STL"/>
+                <mesh filename="package://robot_model/meshes/d435.STL"/>
             </geometry>
             <origin xyz="0 0 0" rpy="1.57 0 -1.57"/>
@@ -251,5 +251,5 @@
         <visual>
             <geometry>
-                <mesh filename="package://urdf_test_node/meshes/t265.STL"/>
+                <mesh filename="package://robot_model/meshes/t265.STL"/>
             </geometry>
             <origin xyz="0 0 0" rpy="1.57 3.14 1.57"/>
@@ -338,5 +338,5 @@
     </transmission>
     <!-- ros2_control configuration for dynamixel_hardware_interface -->
-    <xacro:property name="use_real_hw" value="true"/>
+    <xacro:property name="use_real_hw" value="false"/>
     <xacro:if value="${use_real_hw}">
     <ros2_control name="sekirei_dynamixel_hw" type="system">

Commit message: fix launch

File: ros_ws/src/robot_model/urdf/sekirei_moveit.xacro (robot description, xacro)
@@ -338,5 +338,5 @@
     </transmission>
     <!-- ros2_control configuration for dynamixel_hardware_interface -->
-    <xacro:property name="use_real_hw" value="false"/>
+    <xacro:property name="use_real_hw" value="true"/>
     <xacro:if value="${use_real_hw}">
     <ros2_control name="sekirei_dynamixel_hw" type="system">

Commit message: ???

File: ros_ws/src/robot_model/urdf/sekirei_moveit.xacro (robot description, xacro)
@@ -123,4 +123,5 @@
         </inertial>
     </link>
+    <!-- は？？？ -->
     <joint name="arm_joint3" type="revolute">
         <origin xyz="0.45 0.007 0.084" rpy="0 0 0"/>
@@ -280,4 +281,5 @@
         <type>transmission_interface/SimpleTransmission</type>
         <actuator name="arm_joint1_motor">
+        <!-- 減速比しらべて書く -->
             <mechanicalReduction>1</mechanicalReduction>
             <hardwareInterface>hardware_interface/PositionJointInterface</hardwareInterface>
@@ -338,5 +340,6 @@
     </transmission>
     <!-- ros2_control configuration for dynamixel_hardware_interface -->
-    <xacro:property name="use_real_hw" value="true"/>
+    <!-- Launchファイルから実機制御するかを指定する -->
+    <xacro:property name="use_real_hw" value="$(arg use_real_hw)" />
     <xacro:if value="${use_real_hw}">
     <ros2_control name="sekirei_dynamixel_hw" type="system">
@@ -356,6 +359,8 @@
             <!-- 1:1 mapping: arm_joint1<->dxl21, arm_joint2<->dxl22, ... arm_joint6<->dxl26 (IDs: 21-28, only using 21-26 for 6 joints) -->
             <!-- このへんあやしい -->
-            <param name="joint_to_transmission_matrix">1,0,0,0,0,0, 0,1,0,0,0,0, 0,0,1,0,0,0, 0,0,0,1,0,0, 0,0,0,0,1,0, 0,0,0,0,0,1</param>
-            <param name="transmission_to_joint_matrix">1,0,0,0,0,0, 0,1,0,0,0,0, 0,0,1,0,0,0, 0,0,0,1,0,0, 0,0,0,0,1,0, 0,0,0,0,0,1</param>
+          <!-- Real-hardware mapping: invert joint3 sign so hardware commands/states match URDF orientation
+              Simulation (use_real_hw=false) will keep the identity mapping in its branch. -->
+          <param name="joint_to_transmission_matrix">1,0,0,0,0,0, 0,1,0,0,0,0, 0,0,-1,0,0,0, 0,0,0,1,0,0, 0,0,0,0,1,0, 0,0,0,0,0,1</param>
+          <param name="transmission_to_joint_matrix">1,0,0,0,0,0, 0,1,0,0,0,0, 0,0,-1,0,0,0, 0,0,0,1,0,0, 0,0,0,0,1,0, 0,0,0,0,0,1</param>
         </hardware>
         <!-- Joint configurations -->
@@ -427,4 +432,7 @@
             <param name="Position D Gain">4000</param>
             <param name="Drive Mode">1</param>
+            <!-- ここ反転の可能性大きい -->
+            <!-- やっぱちがうかも -->
+            <!-- 向きは1でそろう -->
         </gpio>
         <gpio name="dxl4">

Commit message: ゼロ補正導入中

File: ros_ws/src/robot_model/urdf/sekirei_moveit.xacro (robot description, xacro)
@@ -130,5 +130,5 @@
         <parent link="arm2_link"/>
         <child link="arm3_link"/>
-        <limit effort="5" lower="0" upper="3.14" velocity="1.571"/>
+        <limit effort="5" lower="-3.14" upper="3.14" velocity="1.571"/>
     </joint>
     <!-- Arm Link 4 -->

Commit message: 減速比対応導入中

File: ros_ws/src/robot_model/urdf/sekirei_moveit.xacro (robot description, xacro)
@@ -127,5 +127,5 @@
     <joint name="arm_joint3" type="revolute">
         <origin xyz="0.45 0.007 0.084" rpy="0 0 0"/>
-        <axis xyz="0 1 0"/>
+        <axis xyz="0 -1 0"/>
         <parent link="arm2_link"/>
         <child link="arm3_link"/>

Commit message: 姿勢とグリッパー開閉同時が実行できたこと確認できた

File: ros_ws/src/robot_model/urdf/sekirei_moveit.xacro (robot description, xacro)
@@ -277,4 +277,20 @@
         <child link="gui_t265_link"/>
     </joint>
+    <link name="gripper_left_link"/>
+    <link name="gripper_right_link"/>
+    <joint name="gripper_joint7" type="revolute">
+    <parent link="arm6_link"/>
+    <child link="gripper_left_link"/>
+    <origin xyz="0 0 0" rpy="0 0 0"/>
+    <axis xyz="0 1 0"/>
+    <limit lower="-1.57" upper="1.57" effort="5" velocity="1.0"/>
+    </joint>
+    <joint name="gripper_joint8" type="revolute">
+    <parent link="arm6_link"/>
+    <child link="gripper_right_link"/>
+    <origin xyz="0 0 0" rpy="0 0 0"/>
+    <axis xyz="0 1 0"/>
+    <limit lower="-1.57" upper="1.57" effort="5" velocity="1.0"/>
+    </joint>
     <!-- transmissions for ros2_control / dynamixel_hardware -->
     <!-- SimpleTransmission used to map actuator to joint -->
@@ -338,4 +354,28 @@
         <joint name="arm_joint6">
             <hardwareInterface>hardware_interface/PositionJointInterface</hardwareInterface>
+        </joint>
+    </transmission>
+    <transmission name="gripper_joint7_trans">
+        <type>transmission_interface/SimpleTransmission</type>
+        <actuator name="gripper_joint7_motor">
+            <mechanicalReduction>1</mechanicalReduction>
+            <hardwareInterface
+            >hardware_interface/PositionJointInterface</hardwareInterface>
+        </actuator>
+        <joint name="gripper_joint7">
+            <hardwareInterface
+            >hardware_interface/PositionJointInterface</hardwareInterface>
+        </joint>
+    </transmission>
+    <transmission name="gripper_joint8_trans">
+        <type>transmission_interface/SimpleTransmission</type>
+        <actuator name="gripper_joint8_motor">
+            <mechanicalReduction>1</mechanicalReduction>
+            <hardwareInterface
+            >hardware_interface/PositionJointInterface</hardwareInterface>
+        </actuator>
+        <joint name="gripper_joint8">
+            <hardwareInterface
+            >hardware_interface/PositionJointInterface</hardwareInterface>
         </joint>
     </transmission>
@@ -352,6 +392,6 @@
             <param name="baud_rate">1000000</param>
             <param name="error_timeout_ms">1000</param>
-            <param name="number_of_joints">6</param>
-            <param name="number_of_transmissions">6</param>
+            <param name="number_of_joints">8</param>
+            <param name="number_of_transmissions">8</param>
             <param name="dynamixel_model_folder">/param/dxl_model</param>
             <param name="disable_torque_at_init">true</param>
@@ -362,6 +402,10 @@
           <!-- Real-hardware mapping: invert joint3 sign so hardware commands/states match URDF orientation
               Simulation (use_real_hw=false) will keep the identity mapping in its branch. -->
-          <param name="joint_to_transmission_matrix">1,0,0,0,0,0, 0,1,0,0,0,0, 0,0,1,0,0,0, 0,0,0,1,0,0, 0,0,0,0,1,0, 0,0,0,0,0,1</param>
-          <param name="transmission_to_joint_matrix">1,0,0,0,0,0, 0,1,0,0,0,0, 0,0,1,0,0,0, 0,0,0,1,0,0, 0,0,0,0,1,0, 0,0,0,0,0,1</param>
+          <param
+                    name="joint_to_transmission_matrix"
+                >1,0,0,0,0,0,0,0, 0,1,0,0,0,0,0,0, 0,0,1,0,0,0,0,0, 0,0,0,1,0,0,0,0, 0,0,0,0,1,0,0,0, 0,0,0,0,0,1,0,0, 0,0,0,0,0,0,1,0, 0,0,0,0,0,0,0,1</param>
+         <param
+                    name="transmission_to_joint_matrix"
+                >1,0,0,0,0,0,0,0, 0,1,0,0,0,0,0,0, 0,0,1,0,0,0,0,0, 0,0,0,1,0,0,0,0, 0,0,0,0,1,0,0,0, 0,0,0,0,0,1,0,0, 0,0,0,0,0,0,1,0, 0,0,0,0,0,0,0,1</param>
         </hardware>
         <!-- Joint configurations -->
@@ -396,4 +440,16 @@
             <state_interface name="velocity"/>
         </joint>
+        <joint name="gripper_joint7">
+            <command_interface name="position" />
+            <state_interface name="position" />
+            <state_interface name="velocity" />
+            <state_interface name="effort" />
+        </joint>
+        <joint name="gripper_joint8">
+            <command_interface name="position" />
+            <state_interface name="position" />
+            <state_interface name="velocity" />
+            <state_interface name="effort" />
+        </joint>
         <!-- GPIO configurations for Dynamixel motors (IDs: 21-26) -->
         <!-- Note: ID 26 is XM430-W350 (model 1020), others are XM540-W270 (model 1120) -->
@@ -468,4 +524,28 @@
             <state_interface name="Present Velocity"/>
             <state_interface name="Present Current"/>
+            <param name="Position P Gain">800</param>
+            <param name="Position I Gain">0</param>
+            <param name="Position D Gain">4000</param>
+            <param name="Drive Mode">0</param>
+        </gpio>
+        <gpio name="dxl7">
+            <param name="type">dxl</param>
+            <param name="ID">27</param>
+            <command_interface name="Goal Position" />
+            <state_interface name="Present Position" />
+            <state_interface name="Present Velocity" />
+            <state_interface name="Present Current" />
+            <param name="Position P Gain">800</param>
+            <param name="Position I Gain">0</param>
+            <param name="Position D Gain">4000</param>
+            <param name="Drive Mode">0</param>
+        </gpio>
+        <gpio name="dxl8">
+            <param name="type">dxl</param>
+            <param name="ID">28</param>
+            <command_interface name="Goal Position" />
+            <state_interface name="Present Position" />
+            <state_interface name="Present Velocity" />
+            <state_interface name="Present Current" />
             <param name="Position P Gain">800</param>
             <param name="Position I Gain">0</param>
@@ -563,4 +643,30 @@
             </state_interface>
         </joint>
+        <joint name="gripper_joint7">
+            <command_interface name="position">
+                <param name="min">-1.57</param>
+                <param name="max">1.57</param>
+            </command_interface>
+            <state_interface name="position">
+                <param name="initial_value">0.0</param>
+            </state_interface>
+            <state_interface name="velocity" />
+            <state_interface name="effort">
+                <param name="initial_value">0.0</param>
+            </state_interface>
+        </joint>
+        <joint name="gripper_joint8">
+            <command_interface name="position">
+                <param name="min">-1.57</param>
+                <param name="max">1.57</param>
+            </command_interface>
+            <state_interface name="position">
+                <param name="initial_value">0.0</param>
+            </state_interface>
+            <state_interface name="velocity" />
+            <state_interface name="effort">
+                <param name="initial_value">0.0</param>
+            </state_interface>
+        </joint>
     </ros2_control>
     </xacro:unless>
